File: Controller/nano.sch (KiCad schematic (older format))
At the start: 25 parts

Commit message: Add nano to main sheet
Connections:
- net labels added: USB_RX, USB_TX
- wire segments 71 -> 73
Other:
- moved on the sheet: D?, R?
Changed lines of the file:
@@
 EESchema Schematic File Version 4
+LIBS:Controller-cache
 EELAYER 29 0
 EELAYER END
@@
 NoConn ~ 5550 1850
 Text Label 4600 1850 0    31   ~ 0
-TX
+USB_TX
 Wire Wire Line
 	4600 1850 4750 1850
 Text Label 4600 1950 0    31   ~ 0
-RX
+USB_RX
 Wire Wire Line
 	4600 1950 4750 1950
-Text Label 9900 3050 0    31   ~ 0
-TX
+Text Label 10150 3050 0    31   ~ 0
+USB_TX
 $Comp
 L Device:C_Small C?
@@
 $EndComp
 Wire Wire Line
-	9400 3050 9500 3050
-Wire Wire Line
-	9800 3050 9850 3050
-Text Label 9900 3150 0    31   ~ 0
-RX
-Wire Wire Line
-	9400 3150 9500 3150
-Wire Wire Line
-	9800 3150 9850 3150
+	10050 3050 10100 3050
+Text Label 10150 3150 0    31   ~ 0
+USB_RX
+Wire Wire Line
+	10050 3150 10100 3150
 Wire Wire Line
 	7350 2150 7500 2150
@@
 5V
 Wire Wire Line
-	9850 2950 9850 3050
-Connection ~ 9850 3050
-Wire Wire Line
-	9850 3050 9900 3050
+	10100 2950 10100 3050
+Connection ~ 10100 3050
+Wire Wire Line
+	10100 3050 10150 3050
 $Comp
 L OPL_Resistor:SMD-RES-1K-1%-1_10W_0603_ R?
 U 1 1 5D4DC1D9
-P 9650 3050
-F 0 "R?" H 9650 3224 45  0000 C CNN
-F 1 "1K" H 9650 3140 45  0000 C CNN
-F 2 "OPL_Resistor:R0603" H 9650 3050 40  0001 C CNN
-F 3 "" H 9650 3050 40  0001 C CNN
-F 4 "RC0603FR-071KL" H 9680 3200 20  0001 C CNN "MPN"
-F 5 "301010298" H 9680 3200 20  0001 C CNN "SKU"
-	1    9650 3050
-	1    0    0    -1
-$EndComp
-Wire Wire Line
-	9850 3250 9850 3150
-Connection ~ 9850 3150
-Wire Wire Line
-	9850 3150 9900 3150
-Text GLabel 10150 2650 2    31   Input ~ 0
+P 9900 3050
+F 0 "R?" H 9900 3224 45  0000 C CNN
+F 1 "1K" H 9900 3140 45  0000 C CNN
+F 2 "OPL_Resistor:R0603" H 9900 3050 40  0001 C CNN
+F 3 "" H 9900 3050 40  0001 C CNN
+F 4 "RC0603FR-071KL" H 9930 3200 20  0001 C CNN "MPN"
+F 5 "301010298" H 9930 3200 20  0001 C CNN "SKU"
+	1    9900 3050
+	1    0    0    -1
+$EndComp
+Wire Wire Line
+	10100 3250 10100 3150
+Connection ~ 10100 3150
+Wire Wire Line
+	10100 3150 10150 3150
+Text GLabel 10400 2650 2    31   Input ~ 0
 5V
-Text GLabel 10150 3550 2    31   Input ~ 0
+Text GLabel 10400 3550 2    31   Input ~ 0
 5V
 $Comp
 L OPL_Optoelectronics:SMD-LED-CLEAR-BLUE_0603_ D?
 U 1 1 5D4DFDA7
-P 9850 2800
-F 0 "D?" V 9808 3002 45  0000 L CNN
-F 1 "LED_BLUE" V 9892 3002 45  0000 L CNN
-F 2 "OPL_Optoelectronics:LED-0603" H 9850 2800 50  0001 C CNN
-F 3 "" H 9850 2800 50  0001 C CNN
-F 4 "19-217-BHC-ZL1M2RY-3T" H 9880 2950 20  0001 C CNN "MPN"
-F 5 "304090045" H 9880 2950 20  0001 C CNN "SKU"
-	1    9850 2800
+P 10100 2800
+F 0 "D?" V 10058 3002 45  0000 L CNN
+F 1 "LED_BLUE" V 10142 3002 45  0000 L CNN
+F 2 "OPL_Optoelectronics:LED-0603" H 10100 2800 50  0001 C CNN
+F 3 "" H 10100 2800 50  0001 C CNN
+F 4 "19-217-BHC-ZL1M2RY-3T" H 10130 2950 20  0001 C CNN "MPN"
+F 5 "304090045" H 10130 2950 20  0001 C CNN "SKU"
+	1    10100 2800
 	0    1    1    0
 $EndComp
@@
 L OPL_Optoelectronics:SMD-LED-CLEAR-BLUE_0603_ D?
 U 1 1 5D4E0FF9
-P 9850 3400
-F 0 "D?" V 9892 3273 45  0000 R CNN
-F 1 "LED_BLUE" V 9808 3273 45  0000 R CNN
-F 2 "OPL_Optoelectronics:LED-0603" H 9850 3400 50  0001 C CNN
-F 3 "" H 9850 3400 50  0001 C CNN
-F 4 "19-217-BHC-ZL1M2RY-3T" H 9880 3550 20  0001 C CNN "MPN"
-F 5 "304090045" H 9880 3550 20  0001 C CNN "SKU"
-	1    9850 3400
+P 10100 3400
+F 0 "D?" V 10142 3273 45  0000 R CNN
+F 1 "LED_BLUE" V 10058 3273 45  0000 R CNN
+F 2 "OPL_Optoelectronics:LED-0603" H 10100 3400 50  0001 C CNN
+F 3 "" H 10100 3400 50  0001 C CNN
+F 4 "19-217-BHC-ZL1M2RY-3T" H 10130 3550 20  0001 C CNN "MPN"
+F 5 "304090045" H 10130 3550 20  0001 C CNN "SKU"
+	1    10100 3400
 	0    -1   -1   0
 $EndComp
@@
 L OPL_Resistor:SMD-RES-220R-5%-1_10W_0603_ R?
 U 1 1 5D4E2240
-P 10000 2650
-F 0 "R?" H 10000 2824 45  0000 C CNN
-F 1 "220R" H 10000 2740 45  0000 C CNN
-F 2 "OPL_Resistor:R0603" H 10000 2736 40  0001 C CNN
-F 3 "" H 10000 2650 40  0001 C CNN
-F 4 "RC0603JR-07220RL" H 10030 2800 20  0001 C CNN "MPN"
-F 5 "301010163" H 10030 2800 20  0001 C CNN "SKU"
-	1    10000 2650
+P 10250 2650
+F 0 "R?" H 10250 2824 45  0000 C CNN
+F 1 "220R" H 10250 2740 45  0000 C CNN
+F 2 "OPL_Resistor:R0603" H 10250 2736 40  0001 C CNN
+F 3 "" H 10250 2650 40  0001 C CNN
+F 4 "RC0603JR-07220RL" H 10280 2800 20  0001 C CNN "MPN"
+F 5 "301010163" H 10280 2800 20  0001 C CNN "SKU"
+	1    10250 2650
 	1    0    0    -1
 $EndComp
@@
 L OPL_Resistor:SMD-RES-1K-1%-1_10W_0603_ R?
 U 1 1 5D4F4CF3
-P 9650 3150
-F 0 "R?" H 9650 3324 45  0000 C CNN
-F 1 "1K" H 9650 3240 45  0000 C CNN
-F 2 "OPL_Resistor:R0603" H 9650 3150 40  0001 C CNN
-F 3 "" H 9650 3150 40  0001 C CNN
-F 4 "RC0603FR-071KL" H 9680 3300 20  0001 C CNN "MPN"
-F 5 "301010298" H 9680 3300 20  0001 C CNN "SKU"
-	1    9650 3150
+P 9900 3150
+F 0 "R?" H 9900 3324 45  0000 C CNN
+F 1 "1K" H 9900 3240 45  0000 C CNN
+F 2 "OPL_Resistor:R0603" H 9900 3150 40  0001 C CNN
+F 3 "" H 9900 3150 40  0001 C CNN
+F 4 "RC0603FR-071KL" H 9930 3300 20  0001 C CNN "MPN"
+F 5 "301010298" H 9930 3300 20  0001 C CNN "SKU"
+	1    9900 3150
 	1    0    0    -1
 $EndComp
@@
 L OPL_Resistor:SMD-RES-220R-5%-1_10W_0603_ R?
 U 1 1 5D4E2F3F
-P 10000 3550
-F 0 "R?" H 10000 3724 45  0000 C CNN
-F 1 "220R" H 10000 3640 45  0000 C CNN
-F 2 "OPL_Resistor:R0603" H 10000 3636 40  0001 C CNN
-F 3 "" H 10000 3550 40  0001 C CNN
-F 4 "RC0603JR-07220RL" H 10030 3700 20  0001 C CNN "MPN"
-F 5 "301010163" H 10030 3700 20  0001 C CNN "SKU"
-	1    10000 3550
+P 10250 3550
+F 0 "R?" H 10250 3724 45  0000 C CNN
+F 1 "220R" H 10250 3640 45  0000 C CNN
+F 2 "OPL_Resistor:R0603" H 10250 3636 40  0001 C CNN
+F 3 "" H 10250 3550 40  0001 C CNN
+F 4 "RC0603JR-07220RL" H 10280 3700 20  0001 C CNN "MPN"
+F 5 "301010163" H 10280 3700 20  0001 C CNN "SKU"
+	1    10250 3550
 	1    0    0    -1
 $EndComp
@@
 Text GLabel 5950 3650 0    31   Input ~ 0
 5V
+Text HLabel 9400 3100 2    39   Output ~ 0
+TX
+Text HLabel 9400 3000 2    39   Input ~ 0
+RX
+Wire Wire Line
+	9400 3100 9400 3150
+Connection ~ 9400 3150
+Wire Wire Line
+	9400 3000 9400 3050
+Connection ~ 9400 3050
+Wire Wire Line
+	9400 3050 9750 3050
+Wire Wire Line
+	9400 3150 9750 3150
 $EndSCHEMATC
