File: Controller/Controller.sch (KiCad schematic (older format))
At the start: 0 parts

Commit message: Almost complete schematic
Parts:
- added C? (x2): 10uF, Capacitor_Tantalum_SMD:CP_EIA-3216-18_Kemet-A, symbol OPL_Capacitor:TANTALUM-SMD-10UF-10V-10%_AVX-A_
- added CN?: SERVO_PWM, OPL_Connector:H3-2.54, symbol OPL_Connector:DIP-BLACK-MALE-HEADER-VERT_3P-2.54_
- added J?: TermAux, TerminalBlock_Phoenix:TerminalBlock_Phoenix_MPT-0,5-4-2.54_1x04_P2.54mm_Horizontal, symbol Connector:Screw_Terminal_01x04
- added J?: TermLaser, TerminalBlock_Phoenix:TerminalBlock_Phoenix_MPT-0,5-4-2.54_1x04_P2.54mm_Horizontal, symbol Connector:Screw_Terminal_01x04
- added J?: LASER_PWR, OPL_Connector:H2-2.54, symbol OPL_Connector:DIP-BLACK-MALE-HEADER-VERT_2P-2.54_
- added J?: LASER_PULSE, OPL_Connector:H2-2.54, symbol OPL_Connector:DIP-BLACK-MALE-HEADER-VERT_2P-2.54_
- added J?: TermLimit, TerminalBlock_Phoenix:TerminalBlock_Phoenix_MPT-0,5-4-2.54_1x04_P2.54mm_Horizontal, symbol Connector:Screw_Terminal_01x04
- added J?: TermControl, TerminalBlock_Phoenix:TerminalBlock_Phoenix_MPT-0,5-4-2.54_1x04_P2.54mm_Horizontal, symbol Connector:Screw_Terminal_01x04
- added J?: TermStop, TerminalBlock_Phoenix:TerminalBlock_Phoenix_MPT-0,5-4-2.54_1x04_P2.54mm_Horizontal, symbol Connector:Screw_Terminal_01x04
- added R?: 10K, OPL_Resistor:R0603, symbol OPL_Resistor:SMD-RES-1K-1%-1_10W_0603_
- added U?: CJ7805, Package_TO_SOT_SMD:TO-252-2, symbol Regulator_Linear:L7805
Connections:
- net HOLD: now also J?.3 (Pin_3)
- net PULSE: now also CN?.1 (P$1), J?.1, J?.3 (Pin_3), R?.2
- net START: now also J?.1 (Pin_1)
- net X_LIMIT: now also J?.1 (Pin_1)
- net Y_LIMIT: now also J?.3 (Pin_3)
- new net 5V: C?.+, CN?.2 (P$2), U?.3 (OUT)
- new net GND: C?.-, C?.-, CN?.3 (P$3), J?.2, J?.2, J?.2 (Pin_2), J?.2 (Pin_2), J?.2 (Pin_2), J?.2 (Pin_2), J?.2 (Pin_2), J?.4 (Pin_4), J?.4 (Pin_4), J?.4 (Pin_4), J?.4 (Pin_4), J?.4 (Pin_4), R?.1, U?.2 (GND)
- new net GRBL_ABORT: J?.1 (Pin_1)
- new net NANO_RESET: J?.3 (Pin_3)
- new net VIN_12V: C?.+, J?.1, J?.1 (Pin_1), J?.1 (Pin_1), J?.3 (Pin_3), U?.1 (IN)
- no-connect marks 8 -> 9
Other:
- note added: "5V Power / 1.5A Max"
- note added: "Accessory Power \n(VIN Only)"
- note added: "Interface Pins"
- note added: "Laser Module Output"
- note added: "Servo Interface"

Commit message: Complete schematic
Parts:
- added J?: PJ-202AH, digikey-footprints:Barrel_Jack_5.5mmODx2.1mmID_PJ-202A, symbol dk_Barrel-Power-Connectors:PJ-202A
Connections:
- net GND: now also J?.2, J?.3
- net VIN_12V: now also J?.1
Other:
- note added: "Power In 12-24V\n(Normally 12V for Laser)"
- moved on the sheet: C?, CN?, J?, R?, U?

Commit message: Set more footprints
Parts:
- gave numbers to parts that had none: 13
Connections:
- no-connect marks 9 -> 6
Changed lines of the file:
@@
 	7650 3750 7550 3750
 NoConn ~ 7650 3050
-NoConn ~ 7650 3350
 NoConn ~ 8350 2850
 NoConn ~ 8350 2950
@@
 	9550 2750 9300 2750
 $Comp
-L Regulator_Linear:L7805 U?
+L Regulator_Linear:L7805 U1
 U 1 1 5D4C3827
 P 2550 2850
-F 0 "U?" H 2550 3092 50  0000 C CNN
+F 0 "U1" H 2550 3092 50  0000 C CNN
 F 1 "CJ7805" H 2550 3001 50  0000 C CNN
 F 2 "Package_TO_SOT_SMD:TO-252-2" H 2575 2700 50  0001 L CIN
@@
 $EndComp
 $Comp
-L power:GND #PWR?
+L power:GND #PWR02
 U 1 1 5D4C4526
 P 2550 3150
-F 0 "#PWR?" H 2550 2900 50  0001 C CNN
+F 0 "#PWR02" H 2550 2900 50  0001 C CNN
 F 1 "GND" H 2555 2977 50  0000 C CNN
 F 2 "" H 2550 3150 50  0001 C CNN
@@
 	1    0    0    -1
 $EndComp
-NoConn ~ 8350 3850
-NoConn ~ 7650 3850
 Text GLabel 3250 2850 2    31   Input ~ 0
 5V
@@
 AR Path="/5D499913/5D4CEFF0" Ref="C?"  Part="1"
 AR Path="/5D4AF8B7/5D4CEFF0" Ref="C?"  Part="1"
-AR Path="/5D4CEFF0" Ref="C?"  Part="1"
-F 0 "C?" V 2908 3128 45  0000 L CNN
+AR Path="/5D4CEFF0" Ref="C2"  Part="1"
+F 0 "C2" V 2908 3128 45  0000 L CNN
 F 1 "10uF" V 2992 3128 45  0000 L CNN
 F 2 "Capacitor_Tantalum_SMD:CP_EIA-3216-18_Kemet-A" H 2950 3000 50  0001 C CNN
@@
 AR Path="/5D499913/5D4D028E" Ref="C?"  Part="1"
 AR Path="/5D4AF8B7/5D4D028E" Ref="C?"  Part="1"
-AR Path="/5D4D028E" Ref="C?"  Part="1"
-F 0 "C?" V 2108 3128 45  0000 L CNN
+AR Path="/5D4D028E" Ref="C1"  Part="1"
+F 0 "C1" V 2108 3128 45  0000 L CNN
 F 1 "10uF" V 2192 3128 45  0000 L CNN
 F 2 "Capacitor_Tantalum_SMD:CP_EIA-3216-18_Kemet-A" H 2150 3000 50  0001 C CNN
@@
 5V Power / 1.5A Max
 $Comp
-L Connector:Screw_Terminal_01x04 J?
+L Connector:Screw_Terminal_01x04 J8
 U 1 1 5D4D369A
 P 5900 3950
-F 0 "J?" H 5818 4267 50  0000 C CNN
+F 0 "J8" H 5818 4267 50  0000 C CNN
 F 1 "TermAux" H 5818 4176 50  0000 C CNN
 F 2 "TerminalBlock_Phoenix:TerminalBlock_Phoenix_MPT-0,5-4-2.54_1x04_P2.54mm_Horizontal" H 5900 3950 50  0001 C CNN
@@
 VIN_12V
 $Comp
-L power:GND #PWR?
+L power:GND #PWR08
 U 1 1 5D4D51CA
 P 6400 3950
-F 0 "#PWR?" H 6400 3700 50  0001 C CNN
+F 0 "#PWR08" H 6400 3700 50  0001 C CNN
 F 1 "GND" V 6405 3822 50  0000 R CNN
 F 2 "" H 6400 3950 50  0001 C CNN
@@
 $EndComp
 $Comp
-L power:GND #PWR?
+L power:GND #PWR09
 U 1 1 5D4D5871
 P 6400 4150
-F 0 "#PWR?" H 6400 3900 50  0001 C CNN
+F 0 "#PWR09" H 6400 3900 50  0001 C CNN
 F 1 "GND" V 6405 4022 50  0000 R CNN
 F 2 "" H 6400 4150 50  0001 C CNN
@@
 AR Path="/5D499913/5D4DCCF3" Ref="R?"  Part="1"
 AR Path="/5D4AF8B7/5D4DCCF3" Ref="R?"  Part="1"
-AR Path="/5D4DCCF3" Ref="R?"  Part="1"
-F 0 "R?" H 7550 4124 45  0000 C CNN
+AR Path="/5D4DCCF3" Ref="R1"  Part="1"
+F 0 "R1" H 7550 4124 45  0000 C CNN
 F 1 "10K" H 7550 4040 45  0000 C CNN
 F 2 "OPL_Resistor:R0603" H 7550 3950 40  0001 C CNN
@@
 	7550 3750 7400 3750
 $Comp
-L power:GND #PWR?
+L power:GND #PWR011
 U 1 1 5D4DDEA4
 P 7550 4100
-F 0 "#PWR?" H 7550 3850 50  0001 C CNN
+F 0 "#PWR011" H 7550 3850 50  0001 C CNN
 F 1 "GND" H 7555 3927 50  0000 C CNN
 F 2 "" H 7550 4100 50  0001 C CNN
@@
 VIN_12V
 $Comp
-L power:GND #PWR?
+L power:GND #PWR04
 U 1 1 5D4DF272
 P 4200 3100
-F 0 "#PWR?" H 4200 2850 50  0001 C CNN
+F 0 "#PWR04" H 4200 2850 50  0001 C CNN
 F 1 "GND" V 4205 2972 50  0000 R CNN
 F 2 "" H 4200 3100 50  0001 C CNN
@@
 $EndComp
 $Comp
-L power:GND #PWR?
+L power:GND #PWR05
 U 1 1 5D4DF278
 P 4200 3300
-F 0 "#PWR?" H 4200 3050 50  0001 C CNN
+F 0 "#PWR05" H 4200 3050 50  0001 C CNN
 F 1 "GND" V 4205 3172 50  0000 R CNN
 F 2 "" H 4200 3300 50  0001 C CNN
@@
 Laser Module Output
 $Comp
-L power:GND #PWR?
+L power:GND #PWR07
 U 1 1 5D4E340E
 P 5300 3650
-F 0 "#PWR?" H 5300 3400 50  0001 C CNN
+F 0 "#PWR07" H 5300 3400 50  0001 C CNN
 F 1 "GND" V 5305 3522 50  0000 R CNN
 F 2 "" H 5300 3650 50  0001 C CNN
@@
 PULSE
 $Comp
-L OPL_Connector:DIP-BLACK-MALE-HEADER-VERT_2P-2.54_ J?
+L OPL_Connector:DIP-BLACK-MALE-HEADER-VERT_2P-2.54_ J5
 U 1 1 5D4EE7E8
 P 4700 3550
-F 0 "J?" H 4592 3904 45  0000 C CNN
+F 0 "J5" H 4592 3904 45  0000 C CNN
 F 1 "LASER_PULSE" H 4592 3820 45  0000 C CNN
 F 2 "OPL_Connector:H2-2.54" H 4700 3550 50  0001 C CNN
@@
 $EndComp
 $Comp
-L OPL_Connector:DIP-BLACK-MALE-HEADER-VERT_2P-2.54_ J?
+L OPL_Connector:DIP-BLACK-MALE-HEADER-VERT_2P-2.54_ J4
 U 1 1 5D4E97DF
 P 4700 2950
-F 0 "J?" H 4592 3304 45  0000 C CNN
+F 0 "J4" H 4592 3304 45  0000 C CNN
 F 1 "LASER_PWR" H 4592 3220 45  0000 C CNN
 F 2 "OPL_Connector:H2-2.54" H 4700 2950 50  0001 C CNN
@@
 	5000 2850 5250 2850
 $Comp
-L power:GND #PWR?
+L power:GND #PWR06
 U 1 1 5D4E3404
 P 5300 3050
-F 0 "#PWR?" H 5300 2800 50  0001 C CNN
+F 0 "#PWR06" H 5300 2800 50  0001 C CNN
 F 1 "GND" V 5305 2922 50  0000 R CNN
 F 2 "" H 5300 3050 50  0001 C CNN
@@
 	5650 2500 3550 2500
 $Comp
-L OPL_Connector:DIP-BLACK-MALE-HEADER-VERT_3P-2.54_ CN?
+L OPL_Connector:DIP-BLACK-MALE-HEADER-VERT_3P-2.54_ CN1
 U 1 1 5D5013A8
 P 6050 2900
-F 0 "CN?" H 5942 3254 45  0000 C CNN
+F 0 "CN1" H 5942 3254 45  0000 C CNN
 F 1 "SERVO_PWM" H 5942 3170 45  0000 C CNN
 F 2 "OPL_Connector:H3-2.54" H 6050 2900 50  0001 C CNN
@@
 5V
 $Comp
-L power:GND #PWR?
+L power:GND #PWR010
 U 1 1 5D502BD0
 P 6450 3050
-F 0 "#PWR?" H 6450 2800 50  0001 C CNN
+F 0 "#PWR010" H 6450 2800 50  0001 C CNN
 F 1 "GND" V 6455 2922 50  0000 R CNN
 F 2 "" H 6450 3050 50  0001 C CNN
@@
 	5800 3550 5800 4250
 $Comp
-L Connector:Screw_Terminal_01x04 J?
+L Connector:Screw_Terminal_01x04 J2
 U 1 1 5D4DF26A
 P 3700 3100
-F 0 "J?" H 3618 3417 50  0000 C CNN
+F 0 "J2" H 3618 3417 50  0000 C CNN
 F 1 "TermLaser" H 3618 3326 50  0000 C CNN
 F 2 "TerminalBlock_Phoenix:TerminalBlock_Phoenix_MPT-0,5-4-2.54_1x04_P2.54mm_Horizontal" H 3700 3100 50  0001 C CNN
@@
 $EndComp
 $Comp
-L Connector:Screw_Terminal_01x04 J?
+L Connector:Screw_Terminal_01x04 J7
 U 1 1 5D512260
 P 5350 4400
-F 0 "J?" V 5350 4600 50  0000 C CNN
+F 0 "J7" V 5350 4600 50  0000 C CNN
 F 1 "TermLimit" V 5450 4350 50  0000 C CNN
 F 2 "TerminalBlock_Phoenix:TerminalBlock_Phoenix_MPT-0,5-4-2.54_1x04_P2.54mm_Horizontal" H 5350 4400 50  0001 C CNN
@@
 $EndComp
 $Comp
-L Connector:Screw_Terminal_01x04 J?
+L Connector:Screw_Terminal_01x04 J6
 U 1 1 5D512CAC
 P 4700 4400
-F 0 "J?" V 4700 4600 50  0000 C CNN
+F 0 "J6" V 4700 4600 50  0000 C CNN
 F 1 "TermControl" V 4800 4350 50  0000 C CNN
 F 2 "TerminalBlock_Phoenix:TerminalBlock_Phoenix_MPT-0,5-4-2.54_1x04_P2.54mm_Horizontal" H 4700 4400 50  0001 C CNN
@@
 HOLD
 $Comp
-L Connector:Screw_Terminal_01x04 J?
+L Connector:Screw_Terminal_01x04 J3
 U 1 1 5D5160BE
 P 4050 4400
-F 0 "J?" V 4050 4600 50  0000 C CNN
+F 0 "J3" V 4050 4600 50  0000 C CNN
 F 1 "TermStop" V 4150 4350 50  0000 C CNN
 F 2 "TerminalBlock_Phoenix:TerminalBlock_Phoenix_MPT-0,5-4-2.54_1x04_P2.54mm_Horizontal" H 4050 4400 50  0001 C CNN
@@
 	5150 4650 4700 4650
 $Comp
-L power:GND #PWR?
+L power:GND #PWR03
 U 1 1 5D5316C3
 P 3750 4650
-F 0 "#PWR?" H 3750 4400 50  0001 C CNN
+F 0 "#PWR03" H 3750 4400 50  0001 C CNN
 F 1 "GND" V 3755 4522 50  0000 R CNN
 F 2 "" H 3750 4650 50  0001 C CNN
@@
 Interface Pins
 $Comp
-L dk_Barrel-Power-Connectors:PJ-202A J?
+L dk_Barrel-Power-Connectors:PJ-202A J1
 U 1 1 5D545F21
 P 2250 4200
-F 0 "J?" H 2183 4425 50  0000 C CNN
+F 0 "J1" H 2183 4425 50  0000 C CNN
 F 1 "PJ-202AH" H 2183 4334 50  0000 C CNN
 F 2 "digikey-footprints:Barrel_Jack_5.5mmODx2.1mmID_PJ-202A" H 2450 4400 60  0001 L CNN
@@
 $EndComp
 $Comp
-L power:GND #PWR?
+L power:GND #PWR01
 U 1 1 5D546925
 P 2350 4400
-F 0 "#PWR?" H 2350 4150 50  0001 C CNN
+F 0 "#PWR01" H 2350 4150 50  0001 C CNN
 F 1 "GND" V 2355 4272 50  0000 R CNN
 F 2 "" H 2350 4400 50  0001 C CNN
@@
 Text Notes 1750 3800 0    59   ~ 0
 Power In 12-24V\n(Normally 12V for Laser)
+$Comp
+L power:PWR_FLAG #FLG0101
+U 1 1 5D584CD1
+P 1450 2600
+F 0 "#FLG0101" H 1450 2675 50  0001 C CNN
+F 1 "PWR_FLAG" H 1450 2773 50  0000 C CNN
+F 2 "" H 1450 2600 50  0001 C CNN
+F 3 "~" H 1450 2600 50  0001 C CNN
+	1    1450 2600
+	1    0    0    -1
+$EndComp
+Text Label 1450 2900 1    31   ~ 0
+VIN_12V
+Wire Wire Line
+	1450 2900 1450 2600
 $EndSCHEMATC

Commit message: Creating Pi layout
Parts:
- added FID1, FID2: Fiducial, Fiducial:Fiducial_1mm_Dia_2mm_Outer, symbol Mechanical:Fiducial
- added H1, H2, H3, H4: Mount, MountingHole:MountingHole_2.5mm_Pad, symbol Mechanical:MountingHole_Pad
- added J9: ConnPi, Connector_PinHeader_2.54mm:PinHeader_1x05_P2.54mm_Vertical, symbol Connector:Conn_01x05_Female
- added R7: 1K, OPL_Resistor:R0603, symbol OPL_Resistor:SMD-RES-1K-1%-1_10W_0603_
- added R8: 2K, OPL_Resistor:R0603, symbol OPL_Resistor:SMD-RES-1K-1%-1_10W_0603_
- C1, C2: symbol OPL_Capacitor:TANTALUM-SMD-10UF-10V-10%_AVX-A_ -> tantalum-smd-10uf-10v-10%_avx-a_:TANTALUM-SMD-10UF-10V-10%_AVX-A_
Connections:
- net 5V: now also C2.1 (+); no longer C2.+
- net GND: now also C1.2 (-), C2.2 (-), H1.1, H2.1, H3.1, H4.1, J9.3 (Pin_3), R8.2; no longer C1.-, C2.-
- net GRBL_RX: now also J9.4 (Pin_4)
- net GRBL_TX: now also R7.1
- net VIN_12V: now also C1.1 (+); no longer C1.+
- new net: J9.5 (Pin_5), R7.2, R8.1
- no-connect marks 6 -> 8
Other:
- note added: "5V"
- note added: "5V <-> 3.3V\nLevel Shift"
- note added: "Gnd"
- note added: "Pi Mounting"
- note added: "Pi RX"
- note added: "Pi Serial Interface"
- note added: "Pi TX"
Changed lines of the file:
@@
 VIN_12V
 $Comp
-L OPL_Capacitor:TANTALUM-SMD-10UF-10V-10%_AVX-A_ C?
+L tantalum-smd-10uf-10v-10%_avx-a_:TANTALUM-SMD-10UF-10V-10%_AVX-A_ C?
 U 1 1 5D4CEFF0
 P 2950 3000
@@
 	2950 2850 3250 2850
 $Comp
-L OPL_Capacitor:TANTALUM-SMD-10UF-10V-10%_AVX-A_ C?
+L tantalum-smd-10uf-10v-10%_avx-a_:TANTALUM-SMD-10UF-10V-10%_AVX-A_ C?
 U 1 1 5D4D028E
 P 2150 3000
@@
 Wire Wire Line
 	1450 2900 1450 2600
+$Comp
+L Mechanical:MountingHole_Pad H2
+U 1 1 5D5AC335
+P 4200 5450
+F 0 "H2" H 4300 5499 50  0000 L CNN
+F 1 "Mount" H 4300 5408 50  0000 L CNN
+F 2 "MountingHole:MountingHole_2.5mm_Pad" H 4200 5450 50  0001 C CNN
+F 3 "~" H 4200 5450 50  0001 C CNN
+	1    4200 5450
+	1    0    0    -1
+$EndComp
+$Comp
+L Mechanical:MountingHole_Pad H3
+U 1 1 5D5AC8F1
+P 4600 5450
+F 0 "H3" H 4700 5499 50  0000 L CNN
+F 1 "Mount" H 4700 5408 50  0000 L CNN
+F 2 "MountingHole:MountingHole_2.5mm_Pad" H 4600 5450 50  0001 C CNN
+F 3 "~" H 4600 5450 50  0001 C CNN
+	1    4600 5450
+	1    0    0    -1
+$EndComp
+$Comp
+L Mechanical:MountingHole_Pad H4
+U 1 1 5D5ACEBA
+P 5000 5450
+F 0 "H4" H 5100 5499 50  0000 L CNN
+F 1 "Mount" H 5100 5408 50  0000 L CNN
+F 2 "MountingHole:MountingHole_2.5mm_Pad" H 5000 5450 50  0001 C CNN
+F 3 "~" H 5000 5450 50  0001 C CNN
+	1    5000 5450
+	1    0    0    -1
+$EndComp
+$Comp
+L Mechanical:MountingHole_Pad H1
+U 1 1 5D5AD190
+P 3800 5450
+F 0 "H1" H 3900 5499 50  0000 L CNN
+F 1 "Mount" H 3900 5408 50  0000 L CNN
+F 2 "MountingHole:MountingHole_2.5mm_Pad" H 3800 5450 50  0001 C CNN
+F 3 "~" H 3800 5450 50  0001 C CNN
+	1    3800 5450
+	1    0    0    -1
+$EndComp
+$Comp
+L power:GND #PWR035
+U 1 1 5D5AFC2D
+P 3750 5550
+F 0 "#PWR035" H 3750 5300 50  0001 C CNN
+F 1 "GND" V 3755 5422 50  0000 R CNN
+F 2 "" H 3750 5550 50  0001 C CNN
+F 3 "" H 3750 5550 50  0001 C CNN
+	1    3750 5550
+	0    1    1    0
+$EndComp
+Wire Wire Line
+	3750 5550 3800 5550
+Wire Wire Line
+	4200 5550 3800 5550
+Connection ~ 3800 5550
+Wire Wire Line
+	4200 5550 4600 5550
+Connection ~ 4200 5550
+Wire Wire Line
+	4600 5550 5000 5550
+Connection ~ 4600 5550
+$Comp
+L Connector:Conn_01x05_Female J9
+U 1 1 5D5B9335
+P 1900 5200
+F 0 "J9" H 1792 5585 50  0000 C CNN
+F 1 "ConnPi" H 1792 5494 50  0000 C CNN
+F 2 "Connector_PinHeader_2.54mm:PinHeader_1x05_P2.54mm_Vertical" H 1900 5200 50  0001 C CNN
+F 3 "~" H 1900 5200 50  0001 C CNN
+	1    1900 5200
+	-1   0    0    -1
+$EndComp
+$Comp
+L power:GND #PWR033
+U 1 1 5D5BC623
+P 2200 5200
+F 0 "#PWR033" H 2200 4950 50  0001 C CNN
+F 1 "GND" V 2205 5072 50  0000 R CNN
+F 2 "" H 2200 5200 50  0001 C CNN
+F 3 "" H 2200 5200 50  0001 C CNN
+	1    2200 5200
+	0    -1   -1   0
+$EndComp
+Wire Wire Line
+	2100 5200 2200 5200
+Text Label 2600 5300 2    31   ~ 0
+GRBL_RX
+Wire Wire Line
+	2600 5300 2100 5300
+Text Label 3050 4900 2    31   ~ 0
+GRBL_TX
+$Comp
+L OPL_Resistor:SMD-RES-1K-1%-1_10W_0603_ R?
+U 1 1 5D5C4586
+P 2800 5250
+AR Path="/5D499913/5D5C4586" Ref="R?"  Part="1"
+AR Path="/5D4AF8B7/5D5C4586" Ref="R?"  Part="1"
+AR Path="/5D5C4586" Ref="R7"  Part="1"
+F 0 "R7" H 2800 5200 45  0000 C CNN
+F 1 "1K" H 2800 5340 45  0000 C CNN
+F 2 "OPL_Resistor:R0603" H 2800 5250 40  0001 C CNN
+F 3 "" H 2800 5250 40  0001 C CNN
+F 4 "RC0603FR-071KL" H 2830 5400 20  0001 C CNN "MPN"
+F 5 "301010298" H 2830 5400 20  0001 C CNN "SKU"
+	1    2800 5250
+	0    1    1    0
+$EndComp
+$Comp
+L OPL_Resistor:SMD-RES-1K-1%-1_10W_0603_ R?
+U 1 1 5D5C71B6
+P 2800 5550
+AR Path="/5D499913/5D5C71B6" Ref="R?"  Part="1"
+AR Path="/5D4AF8B7/5D5C71B6" Ref="R?"  Part="1"
+AR Path="/5D5C71B6" Ref="R8"  Part="1"
+F 0 "R8" H 2800 5500 45  0000 C CNN
+F 1 "2K" H 2800 5640 45  0000 C CNN
+F 2 "OPL_Resistor:R0603" H 2800 5550 40  0001 C CNN
+F 3 "" H 2800 5550 40  0001 C CNN
+F 4 "RC0603FR-072KL" H 2830 5700 20  0001 C CNN "MPN"
+F 5 "301010221" H 2830 5700 20  0001 C CNN "SKU"
+	1    2800 5550
+	0    1    1    0
+$EndComp
+Wire Wire Line
+	2100 5400 2800 5400
+Connection ~ 2800 5400
+Wire Wire Line
+	2800 5100 2800 4900
+Wire Wire Line
+	2800 4900 3050 4900
+$Comp
+L power:GND #PWR034
+U 1 1 5D5CCAC8
+P 2800 5700
+F 0 "#PWR034" H 2800 5450 50  0001 C CNN
+F 1 "GND" V 2805 5572 50  0000 R CNN
+F 2 "" H 2800 5700 50  0001 C CNN
+F 3 "" H 2800 5700 50  0001 C CNN
+	1    2800 5700
+	1    0    0    -1
+$EndComp
+Text Notes 1800 5000 0    31   ~ 0
+5V
+Text Notes 1800 5100 0    31   ~ 0
+5V
+Text Notes 1750 5200 0    31   ~ 0
+Gnd
+Text Notes 1750 5300 0    31   ~ 0
+Pi TX
+Text Notes 1750 5400 0    31   ~ 0
+Pi RX
+Text Notes 2950 5450 0    31   ~ 0
+5V <-> 3.3V\nLevel Shift
+NoConn ~ 2100 5000
+NoConn ~ 2100 5100
+Wire Notes Line
+	1700 4750 3300 4750
+Wire Notes Line
+	3300 4750 3300 6050
+Wire Notes Line
+	3300 6050 1700 6050
+Wire Notes Line
+	1700 6050 1700 4750
+Text Notes 2100 4700 0    59   ~ 0
+Pi Serial Interface
+Wire Notes Line
+	3450 5650 5350 5650
+Wire Notes Line
+	5350 5650 5350 5300
+Wire Notes Line
+	5350 5300 3450 5300
+Wire Notes Line
+	3450 5300 3450 5650
+Text Notes 4150 5250 0    59   ~ 0
+Pi Mounting
+$Comp
+L Mechanical:Fiducial FID1
+U 1 1 5D5E24CD
+P 900 2550
+F 0 "FID1" H 985 2596 50  0000 L CNN
+F 1 "Fiducial" H 985 2505 50  0000 L CNN
+F 2 "Fiducial:Fiducial_1mm_Dia_2mm_Outer" H 900 2550 50  0001 C CNN
+F 3 "~" H 900 2550 50  0001 C CNN
+	1    900  2550
+	1    0    0    -1
+$EndComp
+$Comp
+L Mechanical:Fiducial FID2
+U 1 1 5D5E33A3
+P 900 2750
+F 0 "FID2" H 985 2796 50  0000 L CNN
+F 1 "Fiducial" H 985 2705 50  0000 L CNN
+F 2 "Fiducial:Fiducial_1mm_Dia_2mm_Outer" H 900 2750 50  0001 C CNN
+F 3 "~" H 900 2750 50  0001 C CNN
+	1    900  2750
+	1    0    0    -1
+$EndComp
 $EndSCHEMATC
