File: Controller/Controller.sch (KiCad schematic (older format))
At the start: 22 parts, among them CN1 SERVO_PWM, J1 PJ-202AH, J15 12V_TERM, J2 TermLaser, J3 TermStop, J4 LASER_PWR, J5 LASER_PULSE, J6 TermControl, J7 TermLimit, J8 TermAux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

Commit message: Fixing 10uF caps
Parts:
- C1, C2: footprint Capacitor_Tantalum_SMD:CP_EIA-3216-18_Kemet-A -> OPL_Capacitor:C1206; symbol tantalum-smd-10uf-10v-10%_avx-a_:TANTALUM-SMD-10UF-10V-10%_AVX-A_ -> Device:C; MPN TAJA106K010RNJ -> CC1206KKX5R8BB106; SKU 302020011 -> 302010181
Changed lines of the file:
@@
 VIN_12V
 $Comp
-L tantalum-smd-10uf-10v-10%_avx-a_:TANTALUM-SMD-10UF-10V-10%_AVX-A_ C?
+L Device:C C?
 U 1 1 5D4CEFF0
 P 2950 2950
@@
 AR Path="/5D4AF8B7/5D4CEFF0" Ref="C?"  Part="1"
 AR Path="/5D4CEFF0" Ref="C2"  Part="1"
-F 0 "C2" V 2908 3078 45  0000 L CNN
-F 1 "10uF" V 2992 3078 45  0000 L CNN
-F 2 "Capacitor_Tantalum_SMD:CP_EIA-3216-18_Kemet-A" H 2950 2950 50  0001 C CNN
+F 0 "C2" H 3000 3050 45  0000 L CNN
+F 1 "10uF" H 3050 2950 45  0000 L CNN
+F 2 "OPL_Capacitor:C1206" H 2950 2950 50  0001 C CNN
 F 3 "" H 2950 2950 50  0001 C CNN
-F 4 "TAJA106K010RNJ" H 2980 3100 20  0001 C CNN "MPN"
-F 5 "302020011" H 2980 3100 20  0001 C CNN "SKU"
+F 4 "CC1206KKX5R8BB106" H 2980 3100 20  0001 C CNN "MPN"
+F 5 "302010181" H 2980 3100 20  0001 C CNN "SKU"
 	1    2950 2950
-	0    1    1    0
-$EndComp
-Wire Wire Line
-	1800 2800 2150 2800
-Wire Wire Line
-	2850 2800 2950 2800
-Connection ~ 2950 2800
-Wire Wire Line
-	2950 2800 3250 2800
-$Comp
-L tantalum-smd-10uf-10v-10%_avx-a_:TANTALUM-SMD-10UF-10V-10%_AVX-A_ C?
+	1    0    0    -1
+$EndComp
+$Comp
+L Device:C C?
 U 1 1 5D4D028E
 P 2150 2950
@@
 AR Path="/5D4AF8B7/5D4D028E" Ref="C?"  Part="1"
 AR Path="/5D4D028E" Ref="C1"  Part="1"
-F 0 "C1" V 2108 3078 45  0000 L CNN
-F 1 "10uF" V 2192 3078 45  0000 L CNN
-F 2 "Capacitor_Tantalum_SMD:CP_EIA-3216-18_Kemet-A" H 2150 2950 50  0001 C CNN
+F 0 "C1" H 2200 3050 45  0000 L CNN
+F 1 "10uF" H 2250 2950 45  0000 L CNN
+F 2 "OPL_Capacitor:C1206" H 2150 2950 50  0001 C CNN
 F 3 "" H 2150 2950 50  0001 C CNN
-F 4 "TAJA106K010RNJ" H 2180 3100 20  0001 C CNN "MPN"
-F 5 "302020011" H 2180 3100 20  0001 C CNN "SKU"
+F 4 "CC1206KKX5R8BB106" H 2180 3100 20  0001 C CNN "MPN"
+F 5 "302010181" H 2180 3100 20  0001 C CNN "SKU"
 	1    2150 2950
-	0    -1   1    0
-$EndComp
-Connection ~ 2150 2800
-Wire Wire Line
-	2150 2800 2250 2800
+	-1   0    0    -1
+$EndComp
 Wire Wire Line
 	2150 3100 2550 3100
@@
 Wire Notes Line
 	3100 3700 3100 4350
+Wire Wire Line
+	2850 2800 2950 2800
+Connection ~ 2950 2800
+Wire Wire Line
+	2950 2800 3250 2800
+Wire Wire Line
+	1800 2800 2150 2800
+Connection ~ 2150 2800
+Wire Wire Line
+	2150 2800 2250 2800
 $EndSCHEMATC

Commit message: Add fab files
Parts:
- J2, J3, J6, J7, J8: SKU 320110143 -> 320110118
Changed lines of the file:
@@
 F 2 "TerminalBlock_Phoenix:TerminalBlock_Phoenix_MPT-0,5-4-2.54_1x04_P2.54mm_Horizontal" H 5900 3950 50  0001 C CNN
 F 3 "~" H 5900 3950 50  0001 C CNN
-F 4 "320110143" H 5900 3950 50  0001 C CNN "SKU"
+F 4 "320110118" H 5900 3950 50  0001 C CNN "SKU"
 F 5 "GS019-2.54-04P-5" H 5900 3950 50  0001 C CNN "MPN"
 	1    5900 3950
@@
 F 2 "TerminalBlock_Phoenix:TerminalBlock_Phoenix_MPT-0,5-4-2.54_1x04_P2.54mm_Horizontal" H 3700 3100 50  0001 C CNN
 F 3 "~" H 3700 3100 50  0001 C CNN
-F 4 "320110143" H 3700 3100 50  0001 C CNN "SKU"
+F 4 "320110118" H 3700 3100 50  0001 C CNN "SKU"
 F 5 "GS019-2.54-04P-5" H 3700 3100 50  0001 C CNN "MPN"
 	1    3700 3100
@@
 F 2 "TerminalBlock_Phoenix:TerminalBlock_Phoenix_MPT-0,5-4-2.54_1x04_P2.54mm_Horizontal" H 5350 4400 50  0001 C CNN
 F 3 "~" H 5350 4400 50  0001 C CNN
-F 4 "320110143" H 5350 4400 50  0001 C CNN "SKU"
+F 4 "320110118" H 5350 4400 50  0001 C CNN "SKU"
 F 5 "GS019-2.54-04P-5" H 5350 4400 50  0001 C CNN "MPN"
 	1    5350 4400
@@
 F 2 "TerminalBlock_Phoenix:TerminalBlock_Phoenix_MPT-0,5-4-2.54_1x04_P2.54mm_Horizontal" H 4700 4400 50  0001 C CNN
 F 3 "~" H 4700 4400 50  0001 C CNN
-F 4 "320110143" H 4700 4400 50  0001 C CNN "SKU"
+F 4 "320110118" H 4700 4400 50  0001 C CNN "SKU"
 F 5 "GS019-2.54-04P-5" H 4700 4400 50  0001 C CNN "MPN"
 	1    4700 4400
@@
 F 2 "TerminalBlock_Phoenix:TerminalBlock_Phoenix_MPT-0,5-4-2.54_1x04_P2.54mm_Horizontal" H 4050 4400 50  0001 C CNN
 F 3 "~" H 4050 4400 50  0001 C CNN
-F 4 "320110143" H 4050 4400 50  0001 C CNN "SKU"
+F 4 "320110118" H 4050 4400 50  0001 C CNN "SKU"
 F 5 "GS019-2.54-04P-5" H 4050 4400 50  0001 C CNN "MPN"
 	1    4050 4400
