File: Controller/Controller.kicad_pcb (KiCad board)
At the start: 4 copper layers, 75 x 57 mm, 63 parts, among them CN1 SERVO_PWM, CN10 FEMALE_LEFT, CN11 FEMALE_RIGHT, CN2 CFG1, CN3 CFG1, CN4 CFG1, CN5 FEMALE_LEFT, CN6 FEMALE_RIGHT, CN7 CFG1, CN8 CFG1, CN9 CFG1, J1 PJ-202AH, J10 ICSP, J11 MotorTerm, J12 MotorHeader, J13 MotorTerm, J14 MotorHeader, J15 12V_TERM, J2 TermLaser, J3 TermStop, J4 LASER_PWR, J5 LASER_PULSE, J6 TermControl, J7 TermLimit, J8 TermAux, J9 UJ2-BH-1-TH, K1 SW_RESET, U1 CJ7805, U2 INTERFACE-CH340T_SSOP20_, U3 MCU-ATMEGA328P-AU_TQFP32_, Y1 12MHz, Y2 16MHZ

Commit message: Add fab files
Changed lines of the file:
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@@
     (44 Edge.Cuts user)
     (45 Margin user)
-    (46 B.CrtYd user hide)
+    (46 B.CrtYd user)
     (47 F.CrtYd user)
     (48 B.Fab user)
-    (49 F.Fab user hide)
+    (49 F.Fab user)
   )
   (setup
@@
       (effects (font (size 0.508 0.508) (thickness 0.127)))
     )
-    (fp_text value 1uF (at 0 1.54 90) (layer F.Fab)
+    (fp_text value 1uF (at -3.048 0 90) (layer F.Fab)
       (effects (font (size 1 1) (thickness 0.15)))
     )
@@
       (effects (font (size 0.508 0.508) (thickness 0.127)))
     )
-    (fp_text value 22pF (at 0 1.54 90) (layer F.Fab)
+    (fp_text value 22pF (at 3.429 0 90) (layer F.Fab)
       (effects (font (size 1 1) (thickness 0.15)))
     )
@@
       (effects (font (size 0.508 0.508) (thickness 0.127)))
     )
-    (fp_text value 22pF (at 0 1.54 90) (layer F.Fab)
+    (fp_text value 22pF (at -3.429 0 90) (layer F.Fab)
       (effects (font (size 1 1) (thickness 0.15)))
     )
@@
       (effects (font (size 0.508 0.508) (thickness 0.127)))
     )
-    (fp_text value 1uF (at 0 1.54 90) (layer F.Fab)
+    (fp_text value 1uF (at -2.921 0 90) (layer F.Fab)
       (effects (font (size 1 1) (thickness 0.15)))
     )
@@
       (effects (font (size 0.508 0.508) (thickness 0.127)))
     )
-    (fp_text value LED_BLUE (at 0 1.524 90) (layer F.Fab)
-      (effects (font (size 1 1) (thickness 0.15)))
-    )
-    (fp_text user %R (at 0 -1.525 90) (layer F.Fab)
+    (fp_text value LED_BLUE (at 5.461 0 90) (layer F.Fab) hide
+      (effects (font (size 1 1) (thickness 0.15)))
+    )
+    (fp_text user %R (at 2.413 0 90) (layer F.Fab)
       (effects (font (size 1 1) (thickness 0.15)))
     )
@@
       (effects (font (size 0.508 0.508) (thickness 0.127)))
     )
-    (fp_text value LED_BLUE (at 0 1.524 90) (layer F.Fab)
+    (fp_text value LED_BLUE (at 5.461 0 90) (layer F.Fab) hide
       (effects (font (size 1 1) (thickness 0.15)))
     )
@@
     (fp_line (start 1.393 0.6945) (end -1.393 0.6945) (layer F.CrtYd) (width 0.05))
     (fp_line (start -1.393 0.6945) (end -1.393 -0.6945) (layer F.CrtYd) (width 0.05))
-    (fp_text user %R (at 0 -1.525 90) (layer F.Fab)
+    (fp_text user %R (at 2.54 0 90) (layer F.Fab)
       (effects (font (size 1 1) (thickness 0.15)))
     )
@@
       (effects (font (size 0.508 0.508) (thickness 0.127)))
     )
-    (fp_text value 220R (at 0 1.7 270) (layer F.Fab)
-      (effects (font (size 1 1) (thickness 0.15)))
-    )
-    (fp_text user %R (at 0 -1.5 90) (layer F.Fab)
+    (fp_text value 220R (at 0 1.397 270) (layer F.Fab)
+      (effects (font (size 1 1) (thickness 0.15)))
+    )
+    (fp_text user %R (at 2.54 0 90) (layer F.Fab)
       (effects (font (size 1 1) (thickness 0.15)))
     )
@@
       (effects (font (size 0.508 0.508) (thickness 0.127)))
     )
-    (fp_text value 220R (at 0 1.7 270) (layer F.Fab)
+    (fp_text value 220R (at 0.127 -1.778 270) (layer F.Fab)
       (effects (font (size 1 1) (thickness 0.15)))
     )
@@
     (fp_line (start 0.8 0.4) (end -0.8 0.4) (layer F.Fab) (width 0.1))
     (fp_line (start -0.8 0.4) (end -0.8 -0.4) (layer F.Fab) (width 0.1))
-    (fp_text user %R (at 0 -1.5 90) (layer F.Fab)
+    (fp_text user %R (at 2.54 0 90) (layer F.Fab)
       (effects (font (size 1 1) (thickness 0.15)))
     )
@@
     (tags "THIN PLASIC QUAD FLAT PACKAGE GRID 0.8 MM")
     (attr smd)
-    (fp_text reference U3 (at -4.191 4.064 90) (layer F.SilkS)
+    (fp_text reference U3 (at -0.127 0.127 180) (layer F.SilkS)
       (effects (font (size 0.889 0.889) (thickness 0.1016)))
     )
@@
       (effects (font (size 0.508 0.508) (thickness 0.127)))
     )
-    (fp_text value LED_BLUE (at 0 1.524 90) (layer F.Fab)
+    (fp_text value LED_BLUE (at 5.588 -0.127 90) (layer F.Fab) hide
       (effects (font (size 1 1) (thickness 0.15)))
     )
@@
     (fp_line (start 1.393 0.6945) (end -1.393 0.6945) (layer F.CrtYd) (width 0.05))
     (fp_line (start -1.393 0.6945) (end -1.393 -0.6945) (layer F.CrtYd) (width 0.05))
-    (fp_text user %R (at 0 -1.525 90) (layer F.Fab)
+    (fp_text user %R (at 2.54 -0.127 90) (layer F.Fab)
       (effects (font (size 1 1) (thickness 0.15)))
     )
@@
     (fp_line (start 0.8 0.4) (end -0.8 0.4) (layer F.Fab) (width 0.1))
     (fp_line (start -0.8 0.4) (end -0.8 -0.4) (layer F.Fab) (width 0.1))
-    (fp_text user %R (at 0 -1.5 90) (layer F.Fab)
+    (fp_text user %R (at 2.667 0.127 90) (layer F.Fab)
       (effects (font (size 1 1) (thickness 0.15)))
     )
@@
       (effects (font (size 0.508 0.508) (thickness 0.127)))
     )
-    (fp_text value 10uF (at 0 2.2 90) (layer F.Fab)
-      (effects (font (size 1 1) (thickness 0.15)))
-    )
+    (fp_text value 10uF (at -4.572 2.159 90) (layer F.Fab)
+      (effects (font (size 1 1) (thickness 0.15)))
+    )
