File: Controller/step_driver.sch (KiCad schematic (older format))
At the start: 8 parts, among them CN2 CFG1, CN3 CFG1, CN4 CFG1, CN5 FEMALE_LEFT, CN6 FEMALE_RIGHT, J11 MotorTerm, J12 MotorHeader

Commit message: Add fab files
Parts:
- J11: SKU 320110143 -> 320110118
Changed lines of the file:
@@
 F 2 "TerminalBlock_Phoenix:TerminalBlock_Phoenix_MPT-0,5-4-2.54_1x04_P2.54mm_Horizontal" H 6650 2950 50  0001 C CNN
 F 3 "~" H 6650 2950 50  0001 C CNN
-F 4 "320110143" H 6650 2950 50  0001 C CNN "SKU"
+F 4 "320110118" H 6650 2950 50  0001 C CNN "SKU"
 F 5 "GS019-2.54-04P-5" H 6650 2950 50  0001 C CNN "MPN"
 	1    6650 2950
